Commit message: Update DROK ARM IK autonomous grasp integration

File: src/drok_arm_kinematics/config/drok_arm_kinematics_only.urdf (robot description, URDF)
Before this commit: robot DROK_P_gripper_D405, 12 links, 11 joints
Joints:
- joint GRIPPER_TCP_FIXED_JOINT: origin xyz=0 0 0 rpy=0 0 0 -> xyz=0.05 0 0 rpy=0 0 0
